File: SPI9341/SPI9341/SPI9341.sch (KiCad schematic (older format))
At the start: 4 parts

Commit message: add PIO Unified Debugger
Parts:
- U?: symbol kdn_kicad:LCD_ILI9341_SPI -> SPI9341-rescue:LCD_ILI9341_SPI-kdn_kicad
Changed lines of the file:
@@
 EESchema Schematic File Version 4
+LIBS:SPI9341-cache
 EELAYER 26 0
 EELAYER END
@@
 $EndDescr
 $Comp
-L kdn_kicad:LCD_ILI9341_SPI U?
+L SPI9341-rescue:LCD_ILI9341_SPI-kdn_kicad U?
 U 1 1 5CC9C7CE
 P 5350 2950
